File: breadboard-to-2mm-adapter.sch (KiCad schematic (older format))
At the start: 3 parts, among them P1 CONN_01X40, P2 CONN_02X40, P3 CONN_01X40

Commit message: initial pcb 2x40
Parts:
- P2: footprint (none) -> Pin_Headers_2mm:Pin_Header_Straight_2x40_2mm
Connections:
- net 1 renamed GND
- net 2 renamed VCC
Changed lines of the file:
@@
 F 0 "P2" H 4350 5100 50  0000 C CNN
 F 1 "CONN_02X40" V 4350 3050 50  0000 C CNN
-F 2 "" H 4350 3050 50  0001 C CNN
+F 2 "Pin_Headers_2mm:Pin_Header_Straight_2x40_2mm" H 4350 3050 50  0001 C CNN
 F 3 "" H 4350 3050 50  0000 C CNN
 	1    4350 3050
@@
 	-1   0    0    -1
 $EndComp
+$Comp
+L GND #PWR?
+U 1 1 56C9B43D
+P 2300 1150
+F 0 "#PWR?" H 2300 900 50  0001 C CNN
+F 1 "GND" H 2300 1000 50  0000 C CNN
+F 2 "" H 2300 1150 50  0000 C CNN
+F 3 "" H 2300 1150 50  0000 C CNN
+	1    2300 1150
+	-1   0    0    -1
+$EndComp
+$Comp
+L VCC #PWR?
+U 1 1 56C9B457
+P 6700 1050
+F 0 "#PWR?" H 6700 900 50  0001 C CNN
+F 1 "VCC" H 6700 1200 50  0000 C CNN
+F 2 "" H 6700 1050 50  0000 C CNN
+F 3 "" H 6700 1050 50  0000 C CNN
+	1    6700 1050
+	-1   0    0    -1
+$EndComp
+Wire Wire Line
+	6700 1100 6700 1050
+Wire Wire Line
+	6200 1100 6700 1100
+Wire Wire Line
+	2300 1100 2300 1150
+Wire Wire Line
+	1350 1100 2300 1100
+Text Label 6500 1100 0    60   ~ 0
+2
+Text Label 2100 1100 0    60   ~ 0
+1
+$Comp
+L PWR_FLAG #FLG?
+U 1 1 56C9B635
+P 6200 1050
+F 0 "#FLG?" H 6200 1145 50  0001 C CNN
+F 1 "PWR_FLAG" H 6200 1230 50  0000 C CNN
+F 2 "" H 6200 1050 50  0000 C CNN
+F 3 "" H 6200 1050 50  0000 C CNN
+	1    6200 1050
+	1    0    0    -1
+$EndComp
+Wire Wire Line
+	6200 1050 6200 1100
+$Comp
+L PWR_FLAG #FLG?
+U 1 1 56C9B70A
+P 1350 950
+F 0 "#FLG?" H 1350 1045 50  0001 C CNN
+F 1 "PWR_FLAG" H 1350 1130 50  0000 C CNN
+F 2 "" H 1350 950 50  0000 C CNN
+F 3 "" H 1350 950 50  0000 C CNN
+	1    1350 950
+	1    0    0    -1
+$EndComp
+Wire Wire Line
+	1350 950  1350 1100
 $EndSCHEMATC
